File: vfd_driver.kicad_pcb (KiCad board)
At the start: 2 copper layers, 41.1 x 26.7 mm, 23 parts, among them J1 INPUT, J2 FIL, J3 HV, U1 LM4871, U2 LT1073CS

Commit message: rescue parts
Routing:
- added copper zone on F.Cu, net GND
Changed lines of the file:
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@@
   )
   (setup
-    (last_trace_width 0.508)
+    (last_trace_width 0.25)
     (user_trace_width 0.4064)
     (user_trace_width 0.508)
@@
   (segment (start 60.706 37.719) (end 65.151 37.719) (width 0.508) (layer B.Cu) (net 3) (status 10))
   (segment (start 66.929 39.497) (end 66.929 52.451) (width 0.508) (layer B.Cu) (net 3))
-  (segment (start 39.022 48.006) (end 40.513 48.006) (width 0.508) (layer B.Cu) (net 14) (status 10))
-  (segment (start 41.284 48.777) (end 42.672 48.777) (width 0.508) (layer B.Cu) (net 14) (status 20))
-  (segment (start 40.513 48.006) (end 41.284 48.777) (width 0.508) (layer B.Cu) (net 14))
-  (segment (start 42.672 48.777) (end 43.472 48.777) (width 0.508) (layer B.Cu) (net 14) (status 10))
-  (segment (start 43.481 48.768) (end 44.232 48.768) (width 0.508) (layer B.Cu) (net 14))
-  (segment (start 43.472 48.777) (end 43.481 48.768) (width 0.508) (layer B.Cu) (net 14))
-  (segment (start 45.085 47.915) (end 44.232 48.768) (width 0.508) (layer B.Cu) (net 14))
-  (segment (start 45.085 46.228) (end 45.085 47.915) (width 0.508) (layer B.Cu) (net 14))
-  (segment (start 49.022 46.228) (end 45.085 46.228) (width 0.508) (layer B.Cu) (net 14) (status 10))
   (segment (start 49.403 38.481) (end 49.403 37.846) (width 0.508) (layer B.Cu) (net 3))
   (segment (start 59.398 37.719) (end 60.706 37.719) (width 0.508) (layer B.Cu) (net 3))
@@
   (segment (start 50.927 37.338) (end 53.975 37.338) (width 0.508) (layer B.Cu) (net 3))
   (segment (start 53.975 37.338) (end 55.236 38.599) (width 0.508) (layer B.Cu) (net 3))
-  (segment (start 42.316 42.164) (end 44.323 42.164) (width 0.508) (layer B.Cu) (net 14))
-  (segment (start 45.085 42.926) (end 45.085 46.228) (width 0.508) (layer B.Cu) (net 14))
-  (segment (start 44.323 42.164) (end 45.085 42.926) (width 0.508) (layer B.Cu) (net 14))
   (segment (start 64.135 59.309) (end 62.484 59.309) (width 0.508) (layer B.Cu) (net 4) (status 20))
   (segment (start 64.77 58.674) (end 64.135 59.309) (width 0.508) (layer B.Cu) (net 4))
@@
   (segment (start 31.877 46.736) (end 33.622 46.736) (width 0.508) (layer B.Cu) (net 13) (status 20))
   (segment (start 31.741 46.872) (end 31.877 46.736) (width 0.508) (layer B.Cu) (net 13))
+  (segment (start 39.022 48.006) (end 40.513 48.006) (width 0.508) (layer B.Cu) (net 14) (status 10))
+  (segment (start 41.284 48.777) (end 42.672 48.777) (width 0.508) (layer B.Cu) (net 14) (status 20))
+  (segment (start 40.513 48.006) (end 41.284 48.777) (width 0.508) (layer B.Cu) (net 14))
+  (segment (start 42.672 48.777) (end 43.472 48.777) (width 0.508) (layer B.Cu) (net 14) (status 10))
+  (segment (start 43.481 48.768) (end 44.232 48.768) (width 0.508) (layer B.Cu) (net 14))
+  (segment (start 43.472 48.777) (end 43.481 48.768) (width 0.508) (layer B.Cu) (net 14))
+  (segment (start 45.085 47.915) (end 44.232 48.768) (width 0.508) (layer B.Cu) (net 14))
+  (segment (start 45.085 46.228) (end 45.085 47.915) (width 0.508) (layer B.Cu) (net 14))
+  (segment (start 49.022 46.228) (end 45.085 46.228) (width 0.508) (layer B.Cu) (net 14) (status 10))
+  (segment (start 42.316 42.164) (end 44.323 42.164) (width 0.508) (layer B.Cu) (net 14))
+  (segment (start 45.085 42.926) (end 45.085 46.228) (width 0.508) (layer B.Cu) (net 14))
+  (segment (start 44.323 42.164) (end 45.085 42.926) (width 0.508) (layer B.Cu) (net 14))
   (segment (start 49.022 43.561) (end 49.022 46.228) (width 0.508) (layer B.Cu) (net 14))
   (segment (start 51.943 40.64) (end 49.022 43.561) (width 0.508) (layer B.Cu) (net 14))
@@
     (connect_pads (clearance 0.508))
     (min_thickness 0.254)
+    (fill yes (arc_segments 16) (thermal_gap 0.508) (thermal_bridge_width 0.508))
+    (polygon
+      (pts
+        (xy 27.94 35.56) (xy 68.834 35.56) (xy 68.834 61.976) (xy 27.94 61.976)
+      )
+    )
+  )
+  (zone (net 1) (net_name GND) (layer F.Cu) (hatch edge 0.508)
+    (connect_pads (clearance 0.508))
+    (min_thickness 0.254)
